Commit message: new model with continous joints

File: solidworks/top_assembly_no_gripper_all_continuous/urdf/top_assembly_no_gripper_all_continuous.urdf (robot description, URDF)
Before this commit: robot terp2, 19 links, 18 joints
Links:
- link base_link: geometry collision mesh filename=package://top assembly no gripper all continuous/meshes/bas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; visual mesh filename=package://top assembly no gripper all continuous/meshes/bas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
- link link_arm_1: geometry collision mesh filename=package://top assembly no gripper all continuous/meshes/lin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; visual mesh filename=package://top assembly no gripper all continuous/meshes/lin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
- link link_arm_2: geometry collision mesh filename=package://top assembly no gripper all continuous/meshes/lin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; visual mesh filename=package://top assembly no gripper all continuous/meshes/lin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
- link link_arm_3: geometry collision mesh filename=package://top assembly no gripper all continuous/meshes/lin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; visual mesh filename=package://top assembly no gripper all continuous/meshes/lin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
- link link_arm_4: geometry collision mesh filename=package://top assembly no gripper all continuous/meshes/lin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; visual mesh filename=package://top assembly no gripper all continuous/meshes/lin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
- link link_arm_5: geometry collision mesh filename=package://top assembly no gripper all continuous/meshes/lin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; visual mesh filename=package://top assembly no gripper all continuous/meshes/lin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
- link link_axle: geometry collision mesh filename=package://top assembly no gripper all continuous/meshes/lin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; visual mesh filename=package://top assembly no gripper all continuous/meshes/lin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
- link link_drivewheel_left: geometry collision mesh filename=package://top assembly no gripper all continuous/meshes/lin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; visual mesh filename=package://top assembly no gripper all continuous/meshes/lin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
- link link_drivewheel_right: geometry collision mesh filename=package://top assembly no gripper all continuous/meshes/lin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; visual mesh filename=package://top assembly no gripper all continuous/meshes/lin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
- link link_slot_1: geometry collision mesh filename=package://top assembly no gripper all continuous/meshes/lin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; visual mesh filename=package://top assembly no gripper all continuous/meshes/lin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
- link link_slot_2: geometry collision mesh filename=package://top assembly no gripper all continuous/meshes/lin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; visual mesh filename=package://top assembly no gripper all continuous/meshes/lin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
- link link_slot_3: geometry collision mesh filename=package://top assembly no gripper all continuous/meshes/lin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; visual mesh filename=package://top assembly no gripper all continuous/meshes/lin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
- link link_slot_4: geometry collision mesh filename=package://top assembly no gripper all continuous/meshes/lin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; visual mesh filename=package://top assembly no gripper all continuous/meshes/lin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
- link link_slot_5: geometry collision mesh filename=package://top assembly no gripper all continuous/meshes/lin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; visual mesh filename=package://top assembly no gripper all continuous/meshes/lin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
- link link_slot_6: geometry collision mesh filename=package://top assembly no gripper all continuous/meshes/lin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; visual mesh filename=package://top assembly no gripper all continuous/meshes/lin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
- link link_swivel_back: geometry collision mesh filename=package://top assembly no gripper all continuous/meshes/lin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; visual mesh filename=package://top assembly no gripper all continuous/meshes/lin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
- link link_swivel_front: geometry collision mesh filename=package://top assembly no gripper all continuous/meshes/lin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; visual mesh filename=package://top assembly no gripper all continuous/meshes/lin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
- link link_swivelwheel_back: geometry collision mesh filename=package://top assembly no gripper all continuous/meshes/lin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; visual mesh filename=package://top assembly no gripper all continuous/meshes/lin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
- link link_swivelwheel_front: geometry collision mesh filename=package://top assembly no gripper all continuous/meshes/lin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; visual mesh filename=package://top assembly no gripper all continuous/meshes/lin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
