Commit message: new textbook and paperback URDF

File: solidworks/paperbackURDF/urdf/paperbackURDF.urdf (robot description, URDF)
Before this commit: robot paperback, 1 links, 0 joints
Links:
- link base_link: mass 0.4725 -> 0.0755952272775; geometry collision mesh filename=package://paperbackURDF/meshes/base_link.STL; visual mesh filename=package://paperbackURDF/meshes/base_link.STL

File: solidworks/textbookURDF/urdf/textbookURDF.urdf (robot description, URDF)
Before this commit: robot textbook urdf, 1 links, 0 joints
Links:
- link base_link: mass 3.0845 -> 0.49348564366752; geometry collision mesh filename=package://textbookURDF/meshes/base_link.STL; visual mesh filename=package://textbookURDF/meshes/base_link.STL
