Commit message: added teleop and param control for gripper

File: project2/src/terp2/urdf/terp2_controller.urdf.xacro (robot description, xacro)
@@ -81,4 +81,37 @@
             <state_interface name="velocity" />
         </joint>
+        <!-- Joint Controll for Gripper -->
+        <joint name="joint_gripper_base">
+            <command_interface name="position">
+                <param name="min">-6.283185307</param>
+                <param name="max">6.283185307</param>
+            </command_interface>
+            <state_interface name="position" />
+            <state_interface name="velocity" />
+        </joint>
+        <joint name="joint_gripper_gear">
+            <command_interface name="position">
+                <param name="min">-6.283185307</param>
+                <param name="max">6.283185307</param>
+            </command_interface>
+            <state_interface name="position" />
+            <state_interface name="velocity" />
+        </joint>
+        <joint name="joint_gripper_pad1">
+            <command_interface name="position">
+                <param name="min">-6.283185307</param>
+                <param name="max">6.283185307</param>
+            </command_interface>
+            <state_interface name="position" />
+            <state_interface name="velocity" />
+        </joint>
+        <joint name="joint_gripper_pad2">
+            <command_interface name="position">
+                <param name="min">-6.283185307</param>
+                <param name="max">6.283185307</param>
+            </command_interface>
+            <state_interface name="position" />
+            <state_interface name="velocity" />
+        </joint>
         <!-- REMAINING JOINTS ARE FOR STATE INTERFACES ONLY -->
         <joint name="joint_swivelwheel_front">

Commit message: WIP SLAM

File: project2/src/terp2/urdf/terp2_controller.urdf.xacro (robot description, xacro)
@@ -152,4 +152,5 @@
         </joint>
     </ros2_control>
+        <!-- Put this just after the definition of base_link (but still inside <robot> … </robot>) -->
     <gazebo>
         <plugin filename="libgazebo_ros2_control.so" name="gazebo_ros2_control">

File: project2/src/terp2/urdf/terp2_lidar.urdf.xacro (robot description, xacro)
@@ -7,5 +7,5 @@
   </link>
   <joint name="lidar_joint" type="fixed">
-    <origin xyz="0 0 0.20" rpy="0 0 0"/>
+    <origin xyz="0.1 0 0.20" rpy="0 0 0"/>
     <parent link="base_link"/>
     <child  link="lidar_link"/>
@@ -16,4 +16,6 @@
       <pose>0 0 0 0 0 0</pose>            <!-- relative to lidar_link -->
       <update_rate>10</update_rate>
+      <always_on>true</always_on>
+      <delay>0</delay>
       <ray>
         <scan>
@@ -29,7 +31,9 @@
       <plugin name="gazebo_ros_ray_sensor" filename="libgazebo_ros_ray_sensor.so">
         <ros>
+          <argument>use_sim_time:=true</argument>
           <remapping>~/out:=scan</remapping>   <!-- publishes /scan -->
         </ros>
         <frame_name>lidar_link</frame_name>    <!-- TF frame -->
+         <output_type>sensor_msgs/LaserScan</output_type>
       </plugin>
     </sensor>

File: project2/src/terp2/urdf/terp2_model.urdf.xacro (robot description, xacro)
@@ -45,4 +45,22 @@
     </collision>
   </link>
+    <!-- Put this just after the definition of base_link (but still inside <robot> … </robot>) -->
+  <link name="imu_link"/>
+  <joint name="joint_imu" type="fixed">
+    <parent link="base_link"/>
+    <child  link="imu_link"/>
+  </joint>
+  <gazebo reference="imu_link">
+    <sensor name="terp2_imu" type="imu">
+      <update_rate>100.0</update_rate>
+      <always_on>true</always_on>
+      <plugin name="imu_pub" filename="libgazebo_ros_imu_sensor.so">
+        <ros>
+          <remapping>~/out:=imu</remapping>   <!-- publishes /imu -->
+        </ros>
+        <frame_name>imu_link</frame_name>
+      </plugin>
+    </sensor>
+  </gazebo>
   <link
     name="link_arm_1">
