Commit message: Lidar MVP

File: project2/src/terp2/urdf/terp2_lidar.urdf.xacro (robot description, xacro)
@@ -1,39 +1,37 @@
 <?xml version="1.0"?>
-<!-- ENPM662-Project1-Group1 -->
 <robot name="terp2" xmlns:xacro="http://www.ros.org/wiki/xacro">
-    <gazebo reference="lidar_link">
-        <sensor name="lidar" type="ray">
-            <pose>0.0 0.0 0.1 0 0 0</pose>
-            <always_on>true</always_on>
-            <visualize>true</visualize>
-            <update_rate>5</update_rate>
-            <ray>
-                <scan>
-                    <horizontal>
-                        <samples>360</samples>
-                        <resolution>1.00000</resolution>
-                        <min_angle>0.000000</min_angle>
-                        <max_angle>6.280000</max_angle>
-                    </horizontal>
-                </scan>
-                <range>
-                    <min>0.120000</min>
-                    <max>3.5</max>
-                    <resolution>0.015000</resolution>
-                </range>
-                <noise>
-                    <type>gaussian</type>
-                    <mean>0.0</mean>
-                    <stddev>0.01</stddev>
-                </noise>
-            </ray>
-            <plugin name="scan" filename="libgazebo_ros_ray_sensor.so">
-                <ros>
-                    <remapping>~/out:=scan</remapping>
-                </ros>
-                <output_type>sensor_msgs/LaserScan</output_type>
-                <frame_name>lidar_link</frame_name>
-            </plugin>
-        </sensor>
-    </gazebo>
+  <!-- 1 — mount a tiny, weightless lidar link 20 cm above the base -->
+  <link name="lidar_link">
+    <inertial><mass value="0.01"/><origin xyz="0 0 0"/><inertia
+      ixx="1e-6" iyy="1e-6" izz="1e-6" ixy="0" ixz="0" iyz="0"/></inertial>
+  </link>
+  <joint name="lidar_joint" type="fixed">
+    <origin xyz="0 0 0.20" rpy="0 0 0"/>
+    <parent link="base_link"/>
+    <child  link="lidar_link"/>
+  </joint>
+  <!-- 2 — Gazebo sensor, attached to *lidar_link* -->
+  <gazebo reference="lidar_link">
+    <sensor name="terp2_lidar" type="ray">
+      <pose>0 0 0 0 0 0</pose>            <!-- relative to lidar_link -->
+      <update_rate>10</update_rate>
+      <ray>
+        <scan>
+          <horizontal>
+            <samples>360</samples>
+            <min_angle>-3.14159</min_angle>
+            <max_angle> 3.14159</max_angle>
+          </horizontal>
+        </scan>
+        <range><min>0.12</min><max>12.0</max><resolution>0.01</resolution></range>
+      </ray>
+      <!-- 3 — Gazebo-ROS2 bridge -->
+      <plugin name="gazebo_ros_ray_sensor" filename="libgazebo_ros_ray_sensor.so">
+        <ros>
+          <remapping>~/out:=scan</remapping>   <!-- publishes /scan -->
+        </ros>
+        <frame_name>lidar_link</frame_name>    <!-- TF frame -->
+      </plugin>
+    </sensor>
+  </gazebo>
 </robot>

Commit message: SLAM with issue of hitting us

File: project2/src/terp2/urdf/terp2_lidar.urdf.xacro (robot description, xacro)
@@ -1,5 +1,5 @@
 <?xml version="1.0"?>
 <robot name="terp2" xmlns:xacro="http://www.ros.org/wiki/xacro">
-  <!-- 1 — mount a tiny, weightless lidar link 20 cm above the base -->
+  <!-- Mount weightless lidar link 20cm above the base -->
   <link name="lidar_link">
     <inertial><mass value="0.01"/><origin xyz="0 0 0"/><inertia
@@ -7,9 +7,9 @@
   </link>
   <joint name="lidar_joint" type="fixed">
-    <origin xyz="0.1 0 0.20" rpy="0 0 0"/>
+    <origin xyz="0.72 0.0 0.2" rpy="0 0 0"/>
     <parent link="base_link"/>
     <child  link="lidar_link"/>
   </joint>
-  <!-- 2 — Gazebo sensor, attached to *lidar_link* -->
+  <!-- Attach Gazebo sensor to lidar_link -->
   <gazebo reference="lidar_link">
     <sensor name="terp2_lidar" type="ray">
@@ -26,5 +26,5 @@
           </horizontal>
         </scan>
-        <range><min>0.12</min><max>12.0</max><resolution>0.01</resolution></range>
+        <range><min>0.25</min><max>5.0</max><resolution>0.05</resolution></range>
       </ray>
       <!-- 3 — Gazebo-ROS2 bridge -->

File: project2/src/terp2/urdf/terp2_model.urdf.xacro (robot description, xacro)
@@ -14,8 +14,8 @@
         value="250.0" />
       <inertia
-        ixx="14.0"
+        ixx="4.0"
         ixy="-4.33680868994202E-18"
         ixz="1.11672823766007E-17"
-        iyy="14.0"
+        iyy="4.0"
         iyz="-1.90633701299994E-16"
         izz="8.0" />

Commit message: SLAM seems to be issue with transpose, but algorithm improved

File: project2/src/terp2/urdf/terp2_lidar.urdf.xacro (robot description, xacro)
@@ -7,5 +7,5 @@
   </link>
   <joint name="lidar_joint" type="fixed">
-    <origin xyz="0.72 0.0 0.2" rpy="0 0 0"/>
+    <origin xyz="0.0 0.2 0.32" rpy="0 0 0"/>
     <parent link="base_link"/>
     <child  link="lidar_link"/>
@@ -21,5 +21,5 @@
         <scan>
           <horizontal>
-            <samples>360</samples>
+            <samples>180</samples>
             <min_angle>-3.14159</min_angle>
             <max_angle> 3.14159</max_angle>
