Commit message: trial values for inertia

File: project2/src/terp2/urdf/terp2_model.urdf.xacro (robot description, xacro)
@@ -9,14 +9,14 @@
     <inertial>
       <origin
-        xyz="-2.61923079600778E-19 -0.425995488565801 -4.82390144923432E-18"
-        rpy="0 0 0" />
-      <mass
-        value="90.5491893240932" />
+        xyz="0.0 0.0  -0.4259"
+        rpy="0 0 0" />
+      <mass
+        value="900.5491893240932" />
       <inertia
         ixx="3.48663798151639"
-        ixy="9.85373194917809E-18"
-        ixz="-2.68614302627041E-18"
+        ixy="0.0"
+        ixz="0.0"
         iyy="3.81582853495264"
-        iyz="3.58636747690665E-16"
+        iyz="0.0"
         izz="3.48670868252581" />
     </inertial>
@@ -52,11 +52,11 @@
         rpy="0 0 0" />
       <mass
-        value="0.616850275068085" />
+        value="5.616850275068085" />
       <inertia
         ixx="0.000758328898628989"
         ixy="-0.000117533258784041"
-        ixz="-2.25875452601147E-20"
+        ixz="0.0"
         iyy="0.000758328898628989"
-        iyz="2.25875452601147E-20"
+        iyz="0.0"
         izz="0.000745594953422872" />
     </inertial>
@@ -97,4 +97,5 @@
     <axis
       xyz="0 1 0" />
+    <limit effort="1" velocity="1.57" />
   </joint>
   <link
@@ -108,8 +109,8 @@
       <inertia
         ixx="0.00644980256719211"
-        ixy="-8.68208770935658E-18"
-        ixz="1.35666243727304E-18"
+        ixy="0.0"
+        ixz="0.0"
         iyy="0.439844327950975"
-        iyz="1.08332962219202E-18"
+        iyz="0.0"
         izz="0.439921069814824" />
     </inertial>
@@ -150,4 +151,5 @@
     <axis
       xyz="0 1 0" />
+    <limit effort="1" velocity="1.57" />
   </joint>
   <link
@@ -162,7 +164,7 @@
         ixx="0.00583223984122909"
         ixy="-0.00483062346048854"
-        ixz="-1.96718551825591E-08"
+        ixz="0.0"
         iyy="0.313371733808534"
-        iyz="2.20564241042035E-08"
+        iyz="0.0"
         izz="0.313475132379175" />
     </inertial>
@@ -203,4 +205,5 @@
     <axis
       xyz="0 1 0" />
+    <limit effort="1" velocity="1.57" />
   </joint>
   <link
@@ -211,11 +214,11 @@
         rpy="0 0 0" />
       <mass
-        value="1.25302278742002" />
+        value="10.25302278742002" />
       <inertia
         ixx="0.00143510894590358"
         ixy="-0.000404675486049316"
-        ixz="2.05699952076892E-19"
+        ixz="0.0"
         iyy="0.00413540723242508"
-        iyz="5.74154737412548E-20"
+        iyz="0.0"
         izz="0.00415532866573722" />
     </inertial>
@@ -256,4 +259,5 @@
     <axis
       xyz="0 1 0" />
+    <limit effort="1" velocity="1.57" />
   </joint>
   <link
@@ -264,11 +268,11 @@
         rpy="0 0 0" />
       <mass
-        value="0.616850275068085" />
+        value="5.616850275068085" />
       <inertia
         ixx="0.000758328898628989"
         ixy="0.000117533258784041"
-        ixz="2.25875452601147E-20"
+        ixz="0.0"
         iyy="0.000758328898628989"
-        iyz="4.43552749145502E-20"
+        iyz="0.0"
         izz="0.000745594953422872" />
     </inertial>
@@ -309,4 +313,5 @@
     <axis
       xyz="0 1 0" />
+    <limit effort="1" velocity="1.57" />
   </joint>
   <link
@@ -317,9 +322,9 @@
         rpy="0 0 0" />
       <mass
-        value="0.570999999999999" />
+        value="5.570999999999999" />
       <inertia
         ixx="0.010628303477087"
-        ixy="1.90537446956712E-18"
-        ixz="3.4469644668403E-19"
+        ixy="0.0"
+        ixz="0.0"
         iyy="0.00329411724678925"
         iyz="-0.000203435201401051"
@@ -370,5 +375,5 @@
         rpy="0 0 0" />
       <mass
-        value="0.570999999999999" />
+        value="5.570999999999999" />
       <inertia
         ixx="0.010628303477087"
@@ -423,9 +428,9 @@
         rpy="0 0 0" />
       <mass
-        value="0.571" />
+        value="5.571" />
       <inertia
         ixx="0.010628303477087"
-        ixy="1.23327997120226E-18"
-        ixz="2.60208521396521E-18"
+        ixy="0.0"
+        ixz="0.0"
         iyy="0.00329411724678926"
         iyz="-0.00020343520140105"
@@ -476,9 +481,9 @@
         rpy="0 0 0" />
       <mass
-        value="0.570999999999999" />
+        value="5.570999999999999" />
       <inertia
         ixx="0.010628303477087"
-        ixy="1.13923122087515E-18"
-        ixz="-1.51866403107878E-17"
+        ixy="0.0"
+        ixz="0.0"
         iyy="0.00329411724678926"
         iyz="-0.000203435201401053"
@@ -529,9 +534,9 @@
         rpy="0 0 0" />
       <mass
-        value="0.570999999999999" />
+        value="5.570999999999999" />
       <inertia
         ixx="0.010628303477087"
-        ixy="1.85669622038143E-18"
-        ixz="-2.16840434497101E-19"
+        ixy="0.0"
+        ixz="0.0"
         iyy="0.00329411724678925"
         iyz="-0.000203435201401053"
@@ -582,9 +587,9 @@
         rpy="0 0 0" />
       <mass
-        value="0.570999999999998" />
+        value="5.570999999999998" />
       <inertia
         ixx="0.010628303477087"
-        ixy="2.71050543121376E-19"
-        ixz="8.67361737988404E-19"
+        ixy="0.0"
+        ixz="0.0"
         iyy="0.00329411724678925"
         iyz="-0.000203435201401053"
@@ -635,11 +640,11 @@
         rpy="0 0 0" />
       <mass
-        value="1.62717919613712" />
+        value="6.62717919613712" />
       <inertia
         ixx="0.00105705357324475"
-        ixy="-6.50998919450591E-20"
-        ixz="2.62672673099725E-19"
+        ixy="0.0"
+        ixz="0.0"
         iyy="0.0268955742127174"
-        iyz="3.60636006239083E-21"
+        iyz="0.0"
         izz="0.0271686786600347" />
     </inertial>
@@ -688,11 +693,11 @@
         rpy="0 0 0" />
       <mass
-        value="0.206756066514378" />
+        value="5.206756066514378" />
       <inertia
         ixx="0.000155743535413241"
-        ixy="-2.71050543121376E-20"
-        ixz="9.59505150511326E-20"
+        ixy="0.0"
+        ixz="0.0"
         iyy="0.000155743535413241"
-        iyz="-2.20088256947986E-19"
+        iyz="0.0"
         izz="0.000280473660849326" />
     </inertial>
@@ -741,11 +746,11 @@
         rpy="0 0 0" />
       <mass
-        value="0.206756066514379" />
+        value="5.206756066514379" />
       <inertia
         ixx="0.000155743535413241"
-        ixy="-6.7762635780344E-21"
-        ixz="-1.27691993307046E-19"
+        ixy="0.0"
+        ixz="0.0"
         iyy="0.000155743535413241"
-        iyz="-5.86209497915386E-20"
+        iyz="0.0"
         izz="0.000280473660849326" />
     </inertial>
@@ -794,117 +799,117 @@
         rpy="0 0 0" />
       <mass
-        value="0.0232231111520553" />
+        value="5.0232231111520553" />
+      <inertia
+        ixx="1.33246387076922E-05"
+        ixy="0.0"
+        ixz="0.0"
+        iyy="5.36089786833522E-06"
+        iyz="0.0"
+        izz="1.74288397902587E-05" />
+    </inertial>
+    <visual>
+      <origin
+        xyz="0 0 0"
+        rpy="0 0 0" />
+      <geometry>
+        <mesh
+          filename="package://terp2/meshes/link_swivel_front.STL" />
+      </geometry>
+      <material
+        name="">
+        <color
+          rgba="0.792156862745098 0.819607843137255 0.933333333333333 1" />
+      </material>
+    </visual>
+    <collision>
+      <origin
+        xyz="0 0 0"
+        rpy="0 0 0" />
+      <geometry>
+        <mesh
+          filename="package://terp2/meshes/link_swivel_front.STL" />
+      </geometry>
+    </collision>
+  </link>
+  <joint
+    name="joint_swivel_front"
+    type="continuous">
+    <origin
+      xyz="0 -0.25983 -0.595"
+      rpy="1.5708 0 0" />
+    <parent
+      link="base_link" />
+    <child
+      link="link_swivel_front" />
+    <axis
+      xyz="0 1 0" />
+  </joint>
+  <link
+    name="link_swivelwheel_front">
+    <inertial>
+      <origin
+        xyz="-1.94289029309402E-16 1.99840144432528E-15 -6.44116577227138E-18"
+        rpy="0 0 0" />
+      <mass
+        value="5.104284859690789" />
+      <inertia
+        ixx="4.94884093335827E-05"
+        ixy="0.0"
+        ixz="0.0"
+        iyy="4.94884093335827E-05"
+        iyz="0.0"
+        izz="8.33340897135471E-05" />
+    </inertial>
+    <visual>
+      <origin
+        xyz="0 0 0"
+        rpy="0 0 0" />
+      <geometry>
+        <mesh
+          filename="package://terp2/meshes/link_swivelwheel_front.STL" />
+      </geometry>
+      <material
+        name="">
+        <color
+          rgba="0.792156862745098 0.819607843137255 0.933333333333333 1" />
+      </material>
+    </visual>
+    <collision>
+      <origin
+        xyz="0 0 0"
+        rpy="0 0 0" />
+      <geometry>
+        <mesh
+          filename="package://terp2/meshes/link_swivelwheel_front.STL" />
+      </geometry>
+    </collision>
+  </link>
+  <joint
+    name="joint_swivelwheel_front"
+    type="continuous">
+    <origin
+      xyz="0 -0.0775 0"
+      rpy="-1.5707963267949 -1.3498896571676 1.5707963267949" />
+    <parent
+      link="link_swivel_front" />
+    <child
+      link="link_swivelwheel_front" />
+    <axis
+      xyz="0 0 1" />
+  </joint>
+  <link
+    name="link_swivel_back">
+    <inertial>
+      <origin
+        xyz="0.00751421605065047 -0.0638265063331358 5.55111512312578E-17"
+        rpy="0 0 0" />
+      <mass
+        value="5.0232231111520553" />
       <inertia
         ixx="1.33246387076922E-05"
         ixy="-2.46162177312807E-06"
-        ixz="-1.56492876976418E-22"
+        ixz="0.0"
         iyy="5.36089786833522E-06"
-        iyz="-2.29222280377614E-22"
-        izz="1.74288397902587E-05" />
-    </inertial>
-    <visual>
-      <origin
-        xyz="0 0 0"
-        rpy="0 0 0" />
-      <geometry>
-        <mesh
-          filename="package://terp2/meshes/link_swivel_front.STL" />
-      </geometry>
-      <material
-        name="">
-        <color
-          rgba="0.792156862745098 0.819607843137255 0.933333333333333 1" />
-      </material>
-    </visual>
-    <collision>
-      <origin
-        xyz="0 0 0"
-        rpy="0 0 0" />
-      <geometry>
-        <mesh
-          filename="package://terp2/meshes/link_swivel_front.STL" />
-      </geometry>
-    </collision>
-  </link>
-  <joint
-    name="joint_swivel_front"
-    type="continuous">
-    <origin
-      xyz="0 -0.25983 -0.595"
-      rpy="1.5708 0 0" />
-    <parent
-      link="base_link" />
-    <child
-      link="link_swivel_front" />
-    <axis
-      xyz="0 1 0" />
-  </joint>
-  <link
-    name="link_swivelwheel_front">
-    <inertial>
-      <origin
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
Commit message: better inertia

File: project2/src/terp2/urdf/terp2_model.urdf.xacro (robot description, xacro)
@@ -12,12 +12,12 @@
         rpy="0 0 0" />
       <mass
-        value="52.6261060214922" />
-      <inertia
-        ixx="1.98460895535759"
-        ixy="-4.29338796016744E-18"
-        ixz="1.12118087180101E-17"
-        iyy="1.98464854792286"
-        iyz="-1.90498176028434E-16"
-        izz="2.14793221352269" />
+        value="50.0" />
+      <inertia
+        ixx="50.0"
+        ixy="0.0"
+        ixz="0.0"
+        iyy="50.0"
+        iyz="0.0"
+        izz="100.0" />
     </inertial>
     <visual>
@@ -52,12 +52,12 @@
         rpy="0 0 0" />
       <mass
-        value="1.66549574268383" />
-      <inertia
-        ixx="0.00204748802629827"
-        ixy="-0.00031733979871691"
-        ixz="-6.09863722023096E-20"
-        iyy="0.00204748802629827"
-        iyz="6.09863722023096E-20"
-        izz="0.00201310637424175" />
+        value="1.0" />
+      <inertia
+        ixx="1.0"
+        ixy="0.0"
+        ixz="0.0"
+        iyy="1.0"
+        iyz="0.0"
+        izz="1.0" />
     </inertial>
     <visual>
@@ -105,12 +105,12 @@
         rpy="0 0 0" />
       <mass
-        value="16.2134848604943" />
-      <inertia
-        ixx="0.0174144669314187"
-        ixy="-2.45150223603894E-17"
-        ixz="-2.86226911134673E-16"
-        iyy="1.18757968546763"
-        iyz="1.60167941441756E-18"
-        izz="1.18778688850003" />
+        value="1.0" />
+      <inertia
+        ixx="1.0"
+        ixy="0.0"
+        ixz="0.0"
+        iyy="1.0"
+        iyz="0.0"
+        izz="1.0" />
     </inertial>
     <visual>
@@ -158,12 +158,12 @@
         rpy="0 0 0" />
       <mass
-        value="14.4958805139709" />
-      <inertia
-        ixx="0.0157470475713186"
-        ixy="-0.013042683343319"
-        ixz="-5.31140089477955E-08"
-        iyy="0.846103681283042"
-        iyz="5.95523450835168E-08"
-        izz="0.846382857423772" />
+        value="1.0" />
+      <inertia
+        ixx="1.0"
+        ixy="0.0"
+        ixz="0.0"
+        iyy="1.0"
+        iyz="0.0"
+        izz="1.0" />
     </inertial>
     <visual>
@@ -211,12 +211,12 @@
         rpy="0 0 0" />
       <mass
-        value="3.38316152603405" />
-      <inertia
-        ixx="0.00387479415393967"
-        ixy="-0.00109262381233315"
-        ixz="5.87434023821623E-20"
-        iyy="0.0111655995275477"
-        iyz="6.50336489749628E-20"
-        izz="0.0112193873974905" />
+        value="1.0" />
+      <inertia
+        ixx="1.0"
+        ixy="0.0"
+        ixz="0.0"
+        iyy="1.0"
+        iyz="0.0"
+        izz="1.0" />
     </inertial>
     <visual>
@@ -264,12 +264,12 @@
         rpy="0 0 0" />
       <mass
-        value="1.66549574268383" />
-      <inertia
-        ixx="0.00204748802629827"
-        ixy="0.00031733979871691"
-        ixz="-2.46875710098907E-20"
-        iyy="0.00204748802629827"
-        iyz="2.61953084223851E-20"
-        izz="0.00201310637424175" />
+        value="1.0" />
+      <inertia
+        ixx="1.0"
+        ixy="0.0"
+        ixz="0.0"
+        iyy="1.0"
+        iyz="0.0"
+        izz="1.0" />
     </inertial>
     <visual>
@@ -317,12 +317,12 @@
         rpy="0 0 0" />
       <mass
-        value="4.17469561621429" />
-      <inertia
-        ixx="0.0106568078407958"
-        ixy="6.99602596690303E-19"
-        ixz="-2.02628723288863E-18"
-        iyy="0.0113006453086544"
-        iyz="6.30890306414592E-20"
-        izz="0.0156869078407958" />
+        value="1.0" />
+      <inertia
+        ixx="1.0"
+        ixy="0.0"
+        ixz="0.0"
+        iyy="1.0"
+        iyz="0.0"
+        izz="1.0" />
     </inertial>
     <visual>
@@ -370,12 +370,12 @@
         rpy="0 0 0" />
       <mass
-        value="0.0137837377676252" />
-      <inertia
-        ixx="1.0111387761427E-06"
-        ixy="-2.54599758335775E-26"
-        ixz="6.97933641841617E-22"
-        iyy="1.79254858949165E-06"
-        iyz="7.33453263144415E-23"
-        izz="1.0111387761427E-06" />
+        value="1.0" />
+      <inertia
+        ixx="1.0"
+        ixy="0.0"
+        ixz="0.0"
+        iyy="1.0"
+        iyz="0.0"
+        izz="1.0" />
     </inertial>
     <visual>
@@ -423,12 +423,12 @@
         rpy="0 0 0" />
       <mass
-        value="0.307799999999999" />
-      <inertia
-        ixx="0.000822396019736841"
-        ixy="9.9158388157895E-05"
-        ixz="-4.99588815789484E-06"
-        iyy="0.000259132944078947"
-        iyz="-8.79476151315789E-05"
-        izz="0.000816142944078946" />
+        value="1.0" />
+      <inertia
+        ixx="1.0"
+        ixy="0.0"
+        ixz="0.0"
+        iyy="1.0"
+        iyz="0.0"
+        izz="1.0" />
     </inertial>
     <visual>
@@ -481,12 +481,12 @@
         rpy="0 0 0" />
       <mass
-        value="0.3078" />
-      <inertia
-        ixx="0.000822396019736842"
-        ixy="9.91583881578946E-05"
-        ixz="-4.99588815789472E-06"
-        iyy="0.000259132944078947"
-        iyz="-8.79476151315791E-05"
-        izz="0.000816142944078947" />
+        value="1.0" />
+      <inertia
+        ixx="1.0"
+        ixy="0.0"
+        ixz="0.0"
+        iyy="1.0"
+        iyz="0.0"
+        izz="1.0" />
     </inertial>
     <visual>
@@ -539,12 +539,12 @@
         rpy="0 0 0" />
       <mass
-        value="4.39338382957022" />
-      <inertia
-        ixx="0.00285404464776084"
-        ixy="-1.70250350177076E-19"
-        ixz="7.11884371153108E-19"
-        iyy="0.072618050374337"
-        iyz="-5.27246585089395E-20"
-        izz="0.0733554323820936" />
+        value="5.0" />
+      <inertia
+        ixx="5.0"
+        ixy="0.0"
+        ixz="0.0"
+        iyy="5.0"
+        iyz="0.0"
+        izz="5.0" />
     </inertial>
     <visual>
@@ -592,12 +592,12 @@
         rpy="0 0 0" />
       <mass
-        value="0.558241379588822" />
-      <inertia
-        ixx="0.000420507545615752"
-        ixy="8.59854246748872E-20"
-        ixz="-1.53545401205157E-22"
-        iyy="0.000420507545615752"
-        iyz="-1.39586728368322E-22"
-        izz="0.000757278884293181" />
+        value="20.0" />
+      <inertia
+        ixx="20.0"
+        ixy="0.0"
+        ixz="0.0"
+        iyy="20.0"
+        iyz="0.0"
+        izz="20.0" />
     </inertial>
     <visual>
@@ -645,12 +645,12 @@
         rpy="0 0 0" />
       <mass
-        value="0.558241379588822" />
-      <inertia
-        ixx="0.000420507545615752"
-        ixy="8.59854246748872E-20"
-        ixz="-1.53545401205157E-22"
-        iyy="0.000420507545615752"
-        iyz="-1.39586728368323E-22"
-        izz="0.000757278884293181" />
+        value="20.0" />
+      <inertia
+        ixx="20.0"
+        ixy="0.0"
+        ixz="0.0"
+        iyy="20.0"
+        iyz="0.0"
+        izz="20.0" />
     </inertial>
     <visual>
@@ -698,12 +698,12 @@
         rpy="0 0 0" />
       <mass
-        value="0.0627024001105494" />
-      <inertia
-        ixx="3.59765245107689E-05"
-        ixy="-6.64637878744579E-06"
-        ixz="-4.05272785176755E-22"
-        iyy="1.44744242445051E-05"
-        iyz="-6.32773395706454E-22"
-        izz="4.70578674336986E-05" />
+        value="1.0" />
+      <inertia
+        ixx="1.0"
+        ixy="0.0"
+        ixz="0.0"
+        iyy="1.0"
+        iyz="0.0"
+        izz="1.0" />
     </inertial>
     <visual>
@@ -751,12 +751,12 @@
         rpy="0 0 0" />
       <mass
-        value="0.281569121165131" />
-      <inertia
-        ixx="0.000133618705200673"
-        ixy="2.32062935912338E-20"
-        ixz="5.42345990842091E-21"
-        iyy="0.000133618705200673"
-        iyz="-1.12237552734842E-20"
-        izz="0.000225002042226577" />
+        value="20.0" />
+      <inertia
+        ixx="20.0"
+        ixy="0.0"
+        ixz="0.0"
+        iyy="20.0"
+        iyz="0.0"
+        izz="20.0" />
     </inertial>
     <visual>
@@ -804,12 +804,12 @@
         rpy="0 0 0" />
       <mass
-        value="0.0627024001105494" />
-      <inertia
-        ixx="3.59765245107689E-05"
-        ixy="-6.64637878744579E-06"
-        ixz="-4.21368739414295E-22"
-        iyy="1.44744242445051E-05"
-        iyz="-5.85471765025053E-22"
-        izz="4.70578674336986E-05" />
+        value="1.0" />
+      <inertia
+        ixx="1.0"
+        ixy="0.0"
+        ixz="0.0"
+        iyy="1.0"
+        iyz="0.0"
+        izz="1.0" />
     </inertial>
     <visual>
@@ -857,12 +857,12 @@
         rpy="0 0 0" />
       <mass
-        value="0.281569121165131" />
-      <inertia
-        ixx="0.000133618705200673"
-        ixy="-2.2857326770313E-20"
-        ixz="5.76740160712044E-21"
-        iyy="0.000133618705200673"
-        iyz="-3.28937579428342E-23"
-        izz="0.000225002042226577" />
+        value="20.0" />
+      <inertia
+        ixx="20.0"
+        ixy="0.0"
+        ixz="0.0"
+        iyy="20.0"
+        iyz="0.0"
+        izz="20.0" />
     </inertial>
     <visual>

Commit message: WiP Final

File: project2/src/terp2/urdf/terp2_model.urdf.xacro (robot description, xacro)
@@ -12,10 +12,10 @@
         rpy="0 0 0" />
       <mass
-        value="250.0" />
-      <inertia
-        ixx="4.0"
+        value="300.0" />
+      <inertia
+        ixx="14.0"
         ixy="-4.33680868994202E-18"
         ixz="1.11672823766007E-17"
-        iyy="4.0"
+        iyy="14.0"
         iyz="-1.90633701299994E-16"
         izz="8.0" />
@@ -45,5 +45,4 @@
     </collision>
   </link>
-    <!-- Put this just after the definition of base_link (but still inside <robot> … </robot>) -->
   <link name="imu_link"/>
   <joint name="joint_imu" type="fixed">
